Commit message: 2nd commit

File: description/robot_core.xacro (robot description, xacro)
@@ -1,16 +1,16 @@
 <?xml version="1.0"?>
-<robot xmlns:xacro="http://www.ros.org/wiki/xacro" >
-    <xacro:include filename="inertial_macros.xacro"/>
+<robot xmlns:xacro="http://www.ros.org/wiki/xacro">
+    <xacro:include filename="inertial_macros.xacro" />
     <material name='white'>
-        <color rgba="1 1 1 1"/>
+        <color rgba="1 1 1 1" />
     </material>
     <material name='orange'>
-        <color rgba="1 0.3 0.1 1"/>
+        <color rgba="1 0.3 0.1 1" />
     </material>
     <material name='blue'>
-        <color rgba="0.2 0.2 1 1"/>
+        <color rgba="0.2 0.2 1 1" />
     </material>
     <material name='black'>
-        <color rgba="0 0 0 1"/>
+        <color rgba="0 0 0 1" />
     </material>
     <!-- Base Link -->
@@ -19,11 +19,11 @@
     <!-- Chassis link -->
     <joint name='chassis_joint' type='fixed'>
-        <parent link='base_link'/>
+        <parent link='base_link' />
         <child link='chassis' />
-        <origin xyz='-0.1 0 0'/>
+        <origin xyz='-0.1 0 0' />
     </joint>
     <link name='chassis'>
         <visual>
-            <origin xyz='0.15 0 0.075'/>
+            <origin xyz='0.15 0 0.075' />
             <geometry>
                 <box size="0.3 0.3 0.15" />
@@ -32,5 +32,5 @@
         </visual>
         <collision>
-            <origin xyz='0.15 0 0.075'/>
+            <origin xyz='0.15 0 0.075' />
             <geometry>
                 <box size="0.3 0.3 0.15" />
@@ -38,5 +38,5 @@
         </collision>
         <xacro:inertial_box mass='0.5' x='0.3' y='0.3' z='0.15'>
-            <origin xyz='0.15 0 0.075' rpy='0 0 0'/>
+            <origin xyz='0.15 0 0.075' rpy='0 0 0' />
         </xacro:inertial_box>
     </link>
@@ -44,19 +44,19 @@
     <joint name='left_wheel_joint' type="continuous">
         <parent link='base_link' />
-        <child link='left_wheel'/>
+        <child link='left_wheel' />
         <origin xyz="0 0.175 0" rpy="-${pi/2} 0 0" />
-        <axis xyz="0 0 1"/>
+        <axis xyz="0 0 1" />
     </joint>
-    <link name='left_wheel' >
+    <link name='left_wheel'>
         <visual>
-        <geometry>
-            <cylinder radius='0.05' length='0.04' />
-        </geometry>
-        <material name='blue' />
+            <geometry>
+                <cylinder radius='0.05' length='0.04' />
+            </geometry>
+            <material name='blue' />
         </visual>
         <collision>
-        <geometry>
-            <cylinder radius='0.05' length='0.04' />
-        </geometry>
+            <geometry>
+                <cylinder radius='0.05' length='0.04' />
+            </geometry>
         </collision>
         <xacro:inertial_cylinder mass='0.1' length='0.04' radius='0.5'>
@@ -64,22 +64,22 @@
         </xacro:inertial_cylinder>
     </link>
-        <!-- Right wheel link -->
+    <!-- Right wheel link -->
     <joint name='right_wheel_joint' type="continuous">
         <parent link='base_link' />
-        <child link='right_wheel'/>
+        <child link='right_wheel' />
         <origin xyz="0 -0.175 0" rpy="${pi/2} 0 0" />
-        <axis xyz="0 0 -1"/>
+        <axis xyz="0 0 -1" />
     </joint>
-    <link name='right_wheel' >
+    <link name='right_wheel'>
         <visual>
-        <geometry>
-            <cylinder radius='0.05' length='0.04' />
-        </geometry>
-        <material name='blue' />
+            <geometry>
+                <cylinder radius='0.05' length='0.04' />
+            </geometry>
+            <material name='blue' />
         </visual>
         <collision>
-        <geometry>
-            <cylinder radius='0.05' length='0.04' />
-        </geometry>
+            <geometry>
+                <cylinder radius='0.05' length='0.04' />
+            </geometry>
         </collision>
         <xacro:inertial_cylinder mass='0.1' length='0.04' radius='0.5'>
@@ -89,12 +89,12 @@
     <!-- Caster Wheel -->
     <joint name='caster_wheel_joint' type='fixed'>
-        <parent link='chassis'/>
-        <child link='caster_wheel'/>
-        <origin xyz="0.24 0 0" rpy='0 0 0'/>
+        <parent link='chassis' />
+        <child link='caster_wheel' />
+        <origin xyz="0.24 0 0" rpy='0 0 0' />
     </joint>
     <link name='caster_wheel'>
         <visual>
             <geometry>
-                <sphere radius="0.05"/>
+                <sphere radius="0.05" />
             </geometry>
             <material name='black' />
@@ -102,5 +102,5 @@
         <collision>
             <geometry>
-                <sphere radius="0.05"/>
+                <sphere radius="0.05" />
             </geometry>
         </collision>
