Commit message: 4th commit

File: description/lidar.xacro (robot description, xacro)
@@ -1,5 +1,5 @@
 <?xml version="1.0"?>
 <robot xmlns:xacro="http://www.ros.org/wiki/xacro">
-<xacro:include filename="inertial_macros.xacro" />
+    <xacro:include filename="inertial_macros.xacro" />
     <joint name="laser_joint" type="fixed">
         <parent link="chassis" />
@@ -22,5 +22,5 @@
         </collision>
         <xacro:inertial_cylinder mass="0.1" length="0.04" radius="0.05">
-        <origin xyz="0.1 0 0.175" rpy="0 0 0" />
+            <origin xyz="0.1 0 0.175" rpy="0 0 0" />
         </xacro:inertial_cylinder>
     </link>
@@ -58,3 +58,55 @@
         </sensor>
     </gazebo> -->
+    <!-- Lidar Sensor -->
+    <gazebo>
+        <plugin
+            filename='gz-sim-sensors-system'
+            name='gz::sim::systems::Sensors'>
+            <render_engine>ogre2</render_engine>
+        </plugin>
+    </gazebo>
+    <gazebo reference="laser_frame">
+        <sensor name='gpu_lidar' type='gpu_lidar'>
+            <pose relative_to='laser_frame'>0 0 0 0 0 0</pose>
+            <!--  <topic>scan</topic>
+            <update_rate>5</update_rate>
+            <ros>
+                <argument>~/out:=scan</argument>
+                <frame_id>laser_frame</frame_id>
+            </ros>
+            <output_type>sensor_msgs/LaserScan</output_type>
+        -->
+            <lidar>
+                <scan>
+                    <horizontal>
+                        <samples>2000</samples>
+                        <resolution>1</resolution>
+                        <min_angle>-3.14</min_angle>
+                        <max_angle>3.14</max_angle>
+                    </horizontal>
+                </scan>
+                <range>
+                    <min>0.3</min>
+                    <max>12</max>
+                    <resolution>1</resolution>
+                </range>
+                <noise>
+                    <type>gaussian</type>
+                    <mean>0.0</mean>
+                    <stddev>0.001</stddev>
+                </noise>
+            </lidar>
+            <!-- <gz_frame_id>laser_frame</gz_frame_id> -->
+            <always_on>1</always_on>
+            <visualize>true</visualize>
+            <topic>scan</topic>
+            <update_rate>5</update_rate>
+            <!-- <argument>~/out:=scan</argument>
+                <gz_frame_id>laser_frame</gz_frame_id>
+        -->
+            <frame_id>laser_frame</frame_id>
+            <output_type>sensor_msgs/LaserScan</output_type>
+            <gz_frame_id>laser_frame</gz_frame_id>
+        </sensor>
+    </gazebo>
 </robot>

File: description/robot.urdf.xacro (robot description, xacro)
@@ -1,6 +1,12 @@
 <?xml version="1.0"?>
 <robot xmlns:xacro="http://www.ros.org/wiki/xacro"  name="robot">
+    <xacro:arg name='use_ros2_control' default='true'/>
     <xacro:include filename="robot_core.xacro" />
-    <xacro:include filename="gazebo_control.xacro" />
+    <xacro:if value='$(arg use_ros2_control)'>
+        <xacro:include filename="ros2_control.xacro"/>
+    </xacro:if>
+    <xacro:unless value='$(arg use_ros2_control)'>
+        <xacro:include filename="gazebo_control.xacro" />
+    </xacro:unless>
     <xacro:include filename="lidar.xacro" />
 </robot>

Commit message: SLAM, AMCL, Nav2, Joystick controllable

File: description/lidar.xacro (robot description, xacro)
@@ -25,38 +25,4 @@
         </xacro:inertial_cylinder>
     </link>
-    <!-- <gazebo reference="laser_frame">
-        <plugin
-            filename="gz-sim-sensors-system"
-            name="gz::sim::systems::Sensors">
-            <render_engine>ogre2</render_engine>
-        </plugin>
-        <sensor name="laser" type="gpu_lidar">
-            <plugin
-                filename="gz-sim-sensors-system"
-                name="gz::sim::systems::Sensors">
-                <render_engine>ogre2</render_engine>
-            </plugin>
-            <pose> 0 0 0 0 0 0 </pose>
-            <visualize>true</visualize>
-            <update_rate>10</update_rate>
-            <always_on>true</always_on>
-            <lidar>
-                <scan>
-                    <horizontal>
-                        <samples>360</samples>
-                        <min_angle>-3.14</min_angle>
-                        <max_angle>3.14</max_angle>
-                    </horizontal>
-                </scan>
-                <range>
-                    <min>0.3</min>
-                    <max>12</max>
-                </range>
-            </lidar>
-            <topic>scan</topic>
-            <gz_frame_id>laser_frame</gz_frame_id>
-        </sensor>
-    </gazebo> -->
-    <!-- Lidar Sensor -->
     <gazebo>
         <plugin
@@ -69,12 +35,4 @@
         <sensor name='gpu_lidar' type='gpu_lidar'>
             <pose relative_to='laser_frame'>0 0 0 0 0 0</pose>
-            <!--  <topic>scan</topic>
-            <update_rate>5</update_rate>
-            <ros>
-                <argument>~/out:=scan</argument>
-                <frame_id>laser_frame</frame_id>
-            </ros>
-            <output_type>sensor_msgs/LaserScan</output_type>
-        -->
             <lidar>
                 <scan>
@@ -97,12 +55,8 @@
                 </noise>
             </lidar>
-            <!-- <gz_frame_id>laser_frame</gz_frame_id> -->
             <always_on>1</always_on>
             <visualize>true</visualize>
             <topic>scan</topic>
             <update_rate>5</update_rate>
-            <!-- <argument>~/out:=scan</argument>
-                <gz_frame_id>laser_frame</gz_frame_id>
-        -->
             <frame_id>laser_frame</frame_id>
             <output_type>sensor_msgs/LaserScan</output_type>
@@ -111,2 +65,64 @@
     </gazebo>
 </robot>
+<!--
+<?xml version="1.0"?>
+<robot xmlns:xacro="http://www.ros.org/wiki/xacro">
+    <xacro:include filename="inertial_macros.xacro" />
+    <!Lidar link
+    <link name="laser_frame">
+        <visual>
+            <geometry>
+                <cylinder radius="0.05" length="0.04" />
+            </geometry>
+            <material name="red">
+                <color rgba="1 0 0 1" />
+            </material>
+        </visual>
+        <collision>
+            <geometry>
+                <cylinder radius="0.05" length="0.04" />
+            </geometry>
+        </collision>
+        <xacro:inertial_cylinder mass="0.1" length="0.04" radius="0.05">
+            <origin xyz="0.1 0 0.175" rpy="0 0 0" />
+        </xacro:inertial_cylinder>
+    </link>
+    <!Joint attaching lidar to chassis
+    <joint name="laser_joint" type="fixed">
+        <parent link="chassis"/>
+        <child link="laser_frame"/>
+        <origin xyz="0.1 0 0.175" rpy="0 0 0"/>
+    </joint>
+    <!Gazebo lidar sensor
+    <gazebo reference="laser_frame">
+        <sensor name="gpu_lidar" type="gpu_lidar">
+            <pose relative_to="laser_frame">0 0 0 0 0 0</pose>
+            <lidar>
+                <scan>
+                    <horizontal>
+                        <samples>2000</samples>
+                        <min_angle>-3.14</min_angle>
+                        <max_angle>3.14</max_angle>
+                    </horizontal>
+                </scan>
+                <range>
+                    <min>0.3</min>
+                    <max>12</max>
+                </range>
+                <noise>
+                    <type>gaussian</type>
+                    <mean>0.0</mean>
+                    <stddev>0.001</stddev>
+                </noise>
+            </lidar>
+            <always_on>true</always_on>
+            <visualize>true</visualize>
+            <topic>scan</topic>
+            <update_rate>5</update_rate>
+            <frame_id>laser_frame</frame_id>
+            <output_type>sensor_msgs/LaserScan</output_type>
+            <gz_frame_id>laser_frame</gz_frame_id>
+        </sensor>
+    </gazebo>
+</robot>
+-->

File: description/robot.urdf.xacro (robot description, xacro)
@@ -9,4 +9,5 @@
         <xacro:include filename="gazebo_control.xacro" />
     </xacro:unless>
-    <xacro:include filename="lidar.xacro" />
+    <!-- <xacro:include filename="lidar.xacro" /> -->
+    <xacro:include filename="demo.lidar.xacro" />
 </robot>
