Commit message: Drivable on Real Robot, Lidar not attached

File: description/robot.urdf.xacro (robot description, xacro)
@@ -2,4 +2,5 @@
 <robot xmlns:xacro="http://www.ros.org/wiki/xacro"  name="robot">
     <xacro:arg name='use_ros2_control' default='true'/>
+    <xacro:arg name='sim_mode' default='false'/>
     <xacro:include filename="robot_core.xacro" />
     <xacro:if value='$(arg use_ros2_control)'>

File: description/ros2_control.xacro (robot description, xacro)
@@ -1,4 +1,37 @@
 <?xml version="1.0"?>
 <robot xmlns:xacro="http://www.ros.org/wiki/xacro">
+    <xacro:unless value='$(arg sim_mode)'>
+    <ros2_control name="RealRobot" type="system">
+       <hardware>
+          <plugin>diffdrive_arduino/DiffDriveAuduinoHardware</plugin>
+          <param name="example_param_hw_start_duration_sec">0</param>
+          <param name="example_param_hw_stop_duration_sec">3.0</param>
+          <param name="left_wheel_name">left_wheel_joint</param>
+          <param name="right_wheel_name">right_wheel_joint</param>
+          <param name="loop_rate">10</param>
+          <param name="device">/dev/ttyACM0</param>
+          <param name="baud_rate">57600</param>
+          <param name="timeout_ms">1000</param>
+          <param name="enc_counts_per_rev">8800</param>
+        </hardware>
+        <joint name='left_wheel_joint'>
+            <command_interface name='velocity'>
+                <param name='min'>-10</param>
+                <param name='max'>10</param>
+            </command_interface>
+            <state_interface name='position'/>
+            <state_interface name='velocity'/>
+        </joint>
+         <joint name='right_wheel_joint'>
+            <command_interface name='velocity'>
+                <param name='min'>-10</param>
+                <param name='max'>10</param>
+            </command_interface>
+            <state_interface name='position'/>
+            <state_interface name='velocity'/>
+        </joint>
+    </ros2_control>
+    </xacro:unless>
+    <xacro:if value='$(arg sim_mode)'>
     <ros2_control name="GazeboSimSystem" type="system">
         <hardware>
@@ -22,9 +55,11 @@
         </joint>
     </ros2_control>
-    <gazebo>
+    </xacro:if>
+   <!--<gazebo>
         <plugin name="gz_ros2_control::GazeboSimROS2ControlPlugin"
             filename="libgz_ros2_control-system.so">
             <parameters>$(find my_bot_one)/config/my_controllers.yaml</parameters>
+            <parameters>$(find my_bot_one)/config/gaz_ros2_ctl_use_sim.yaml</parameters>
         </plugin>
-    </gazebo>
+    </gazebo> -->
 </robot>
