Commit message: Change package name my_bot_one to autonomous_waitress_robot. URDF adjusted. New world created.

File: description/gazebo_control.xacro (robot description, xacro)
@@ -7,6 +7,6 @@
             <left_joint>left_wheel_joint</left_joint>
             <right_joint>right_wheel_joint</right_joint>
-            <wheel_separation>0.35</wheel_separation>
-            <wheel_radius>0.05</wheel_radius>
+            <wheel_separation>0.292</wheel_separation>
+            <wheel_radius>0.031</wheel_radius>
             <!-- Limit -->
             <max_linear_acceleration>10</max_linear_acceleration>
@@ -44,12 +44,4 @@
         <sensor name='gpu_lidar' type='gpu_lidar'>
             <pose relative_to='laser_frame'>0 0 0 0 0 0</pose>
-            <!--  <topic>scan</topic>
-            <update_rate>5</update_rate>
-            <ros>
-                <argument>~/out:=scan</argument>
-                <frame_id>laser_frame</frame_id>
-            </ros>
-            <output_type>sensor_msgs/LaserScan</output_type>
-        -->
             <lidar>
                 <scan>

File: description/robot.urdf.xacro (robot description, xacro)
@@ -2,5 +2,5 @@
 <robot xmlns:xacro="http://www.ros.org/wiki/xacro"  name="robot">
     <xacro:arg name='use_ros2_control' default='true'/>
-    <xacro:arg name='sim_mode' default='false'/>
+    <xacro:arg name='sim_mode' default='true'/>
     <xacro:include filename="robot_core.xacro" />
     <xacro:if value='$(arg use_ros2_control)'>

File: description/robot_core.xacro (robot description, xacro)
@@ -19,4 +19,5 @@
     <!-- Base Link -->
     <link name="base_link">
+        <origin xyz='0 0 0' rpy='0 0 0'/>
     </link>
     <!-- Base Footprint Link -->
@@ -56,5 +57,5 @@
         <parent link="base_link" />
         <child link="left_wheel" />
-        <origin xyz="0 0.175 0" rpy="-${pi/2} 0 0" />
+        <origin xyz="0 0.146 0" rpy="-${pi/2} 0 0" />
         <axis xyz="0 0 1" />
         <limit effort="0.05" velocity="10.0" />
@@ -69,8 +70,8 @@
         <collision>
             <geometry>
-                <sphere radius="0.05" />
+                <sphere radius="0.031" />
             </geometry>
         </collision>
-        <xacro:inertial_cylinder mass="0.1" length="0.04" radius="0.05">
+        <xacro:inertial_cylinder mass="0.1" length="0.04" radius="0.031">
             <origin xyz="0 0 0" rpy="0 0 0" />
         </xacro:inertial_cylinder>
@@ -80,5 +81,5 @@
         <parent link="base_link" />
         <child link="right_wheel" />
-        <origin xyz="0 -0.175 0" rpy="${pi/2} 0 0" />
+        <origin xyz="0 -0.146 0" rpy="${pi/2} 0 0" />
         <axis xyz="0 0 -1" />
         <limit effort="0.05" velocity="10.0" />
@@ -93,8 +94,8 @@
         <collision>
             <geometry>
-                <sphere radius="0.05" />
+                <sphere radius="0.031" />
             </geometry>
         </collision>
-        <xacro:inertial_cylinder mass="0.1" length="0.04" radius="0.05">
+        <xacro:inertial_cylinder mass="0.1" length="0.04" radius="0.031">
             <origin xyz="0 0 0" rpy="0 0 0" />
         </xacro:inertial_cylinder>
@@ -115,8 +116,8 @@
         <collision>
             <geometry>
-                <sphere radius="0.05" />
+                <sphere radius="0.031" />
             </geometry>
         </collision>
-        <xacro:inertial_sphere mass="0.1" radius="0.05">
+        <xacro:inertial_sphere mass="0.1" radius="0.031">
             <origin xyz="0 0 0" rpy="0 0 0" />
         </xacro:inertial_sphere>

File: description/ros2_control.xacro (robot description, xacro)
@@ -2,64 +2,64 @@
 <robot xmlns:xacro="http://www.ros.org/wiki/xacro">
     <xacro:unless value='$(arg sim_mode)'>
-    <ros2_control name="RealRobot" type="system">
-       <hardware>
-          <plugin>diffdrive_arduino/DiffDriveAuduinoHardware</plugin>
-          <param name="example_param_hw_start_duration_sec">0</param>
-          <param name="example_param_hw_stop_duration_sec">3.0</param>
-          <param name="left_wheel_name">left_wheel_joint</param>
-          <param name="right_wheel_name">right_wheel_joint</param>
-          <param name="loop_rate">10</param>
-          <param name="device">/dev/ttyACM0</param>
-          <param name="baud_rate">57600</param>
-          <param name="timeout_ms">1000</param>
-          <param name="enc_counts_per_rev">8800</param>
-        </hardware>
-        <joint name='left_wheel_joint'>
-            <command_interface name='velocity'>
-                <param name='min'>-10</param>
-                <param name='max'>10</param>
-            </command_interface>
-            <state_interface name='position'/>
-            <state_interface name='velocity'/>
-        </joint>
-         <joint name='right_wheel_joint'>
-            <command_interface name='velocity'>
-                <param name='min'>-10</param>
-                <param name='max'>10</param>
-            </command_interface>
-            <state_interface name='position'/>
-            <state_interface name='velocity'/>
-        </joint>
-    </ros2_control>
+        <ros2_control name="RealRobot" type="system">
+            <hardware>
+                <plugin>diffdrive_arduino/DiffDriveAuduinoHardware</plugin>
+                <param name="example_param_hw_start_duration_sec">0</param>
+                <param name="example_param_hw_stop_duration_sec">3.0</param>
+                <param name="left_wheel_name">left_wheel_joint</param>
+                <param name="right_wheel_name">right_wheel_joint</param>
+                <param name="loop_rate">10</param>
+                <param name="device">/dev/ttyACM0</param>
+                <param name="baud_rate">57600</param>
+                <param name="timeout_ms">1000</param>
+                <param name="enc_counts_per_rev">8800</param>
+            </hardware>
+            <joint name='left_wheel_joint'>
+                <command_interface name='velocity'>
+                    <param name='min'>-10</param>
+                    <param name='max'>10</param>
+                </command_interface>
+                <state_interface name='position' />
+                <state_interface name='velocity' />
+            </joint>
+            <joint name='right_wheel_joint'>
+                <command_interface name='velocity'>
+                    <param name='min'>-10</param>
+                    <param name='max'>10</param>
+                </command_interface>
+                <state_interface name='position' />
+                <state_interface name='velocity' />
+            </joint>
+        </ros2_control>
     </xacro:unless>
-    <xacro:if value='$(arg sim_mode)'>
-    <ros2_control name="GazeboSimSystem" type="system">
-        <hardware>
-            <plugin>gz_ros2_control/GazeboSimSystem</plugin>
-        </hardware>
-        <joint name='left_wheel_joint'>
-            <command_interface name='velocity'>
-                <param name='min'>-10</param>
-                <param name='max'>10</param>
-            </command_interface>
-            <state_interface name='velocity'/>
-            <state_interface name='position'/>
-        </joint>
-         <joint name='right_wheel_joint'>
-            <command_interface name='velocity'>
-                <param name='min'>-10</param>
-                <param name='max'>10</param>
-            </command_interface>
-            <state_interface name='velocity'/>
-            <state_interface name='position'/>
-        </joint>
-    </ros2_control>
+    <xacro:if value="$(arg sim_mode)">
+        <ros2_control name="GazeboSimSystem" type="system">
+            <hardware>
+                <plugin>gz_ros2_control/GazeboSimSystem</plugin>
+            </hardware>
+            <joint name="left_wheel_joint">
+                <command_interface name="velocity">
+                    <param name="min">-10</param>
+                    <param name="max">10</param>
+                </command_interface>
+                <state_interface name="position" />
+                <state_interface name="velocity" />
+            </joint>
+            <joint name="right_wheel_joint">
+                <command_interface name="velocity">
+                    <param name="min">-10</param>
+                    <param name="max">10</param>
+                </command_interface>
+                <state_interface name="position" />
+                <state_interface name="velocity" />
+            </joint>
+        </ros2_control>
     </xacro:if>
-   <!--<gazebo>
+    <gazebo>
         <plugin name="gz_ros2_control::GazeboSimROS2ControlPlugin"
             filename="libgz_ros2_control-system.so">
-            <parameters>$(find my_bot_one)/config/my_controllers.yaml</parameters>
-            <parameters>$(find my_bot_one)/config/gaz_ros2_ctl_use_sim.yaml</parameters>
+            <parameters>$(find autonomous_waitress_robot)/config/my_controllers.yaml</parameters>
+            <parameters>$(find autonomous_waitress_robot)/config/gaz_ros2_ctl_use_sim.yaml</parameters>
         </plugin>
-    </gazebo> -->
+    </gazebo>
 </robot>
